Commit message: arm.xacro ではアーム3リンクの visual と関節基本情報まで構成

File: src/my_robot_description/urdf/common_properties.xacro (robot description, xacro)
@@ -6,4 +6,10 @@
     <material name="grey">
         <color rgba="0.5 0.5 0.5 1"/>
+    </material>
+    <material name="orange">
+        <color rgba="1.0 0.5 0 1"/>
+    </material>
+    <material name="yellow">
+        <color rgba="1.0 1.0 0 1"/>
     </material>
     <xacro:macro name="box_inertia" params="m x y z o_xyz o_rpy">
