Commit message: add arm joint control topics to spawn to gazeo

File: src/my_robot_description/urdf/arm.xacro (robot description, xacro)
@@ -16,4 +16,12 @@
             <material name="orange" />
         </visual>
+        <collision>
+         <geometry>
+            <box size="${arm_base_length} ${arm_base_width} ${arm_base_height}" />
+            </geometry>
+            <origin xyz="0 0 ${arm_base_height / 2.0}" rpy="0 0 0" />
+        </collision>
+        <xacro:box_inertia m="5.0" x="${arm_base_length}" y="${arm_base_width}" z="${arm_base_height}"
+                           o_xyz="0 0 ${arm_base_height / 2.0}" o_rpy="0 0 0" />
     </link>
     <link name="forearm_link">
@@ -25,4 +33,12 @@
             <material name="yellow" />
         </visual>
+        <collision>
+            <geometry>
+            <cylinder radius="${forearm_radius}" length="${forearm_length}" />
+            </geometry>
+            <origin xyz="0 0 ${forearm_length / 2.0}" rpy="0 0 0" />
+        </collision>
+        <xacro:cylinder_inertia m="0.3" r="${forearm_radius}" l="${forearm_length}"
+                                o_xyz="0 0 ${forearm_length / 2.0}" o_rpy="0 0 0" />
     </link>
     <link name="hand_link">
@@ -34,4 +50,12 @@
             <material name="orange" />
         </visual>
+        <collision>
+        <geometry>
+            <cylinder radius="${hand_radius}" length="${hand_length}" />
+            </geometry>
+            <origin xyz="0 0 ${hand_length / 2.0}" rpy="0 0 0" />
+        </collision>
+        <xacro:cylinder_inertia m="0.3" r="${hand_radius}" l="${hand_length}"
+                                o_xyz="0 0 ${hand_length / 2.0}" o_rpy="0 0 0" />
     </link>
     <joint name="arm_base_foream_joint" type="revolute">
@@ -41,4 +65,5 @@
         <axis xyz="0 1 0" />
         <limit lower="0" upper="${pi/2}" effort="100" velocity="100" />
+        <dynamics friction="0.3" damping="0.3" />
     </joint>
     <joint name="forearm_hand_joint" type="revolute">
@@ -48,4 +73,5 @@
         <axis xyz="0 1 0" />
         <limit lower="0" upper="${pi/2}" effort="100" velocity="100" />
+        <dynamics friction="0.3" damping="0.3" />
     </joint>
 </robot>

File: src/my_robot_description/urdf/standalone_arm.urdf.xacro (robot description, xacro)
@@ -3,3 +3,4 @@
     <xacro:include filename="common_properties.xacro" />
     <xacro:include filename="arm.xacro" />
+    <xacro:include filename="arm_gazebo.xacro" />
 </robot>

Commit message: Project: add a robot arm on top of the robot

File: src/my_robot_description/urdf/arm.xacro (robot description, xacro)
@@ -22,5 +22,5 @@
             <origin xyz="0 0 ${arm_base_height / 2.0}" rpy="0 0 0" />
         </collision>
-        <xacro:box_inertia m="5.0" x="${arm_base_length}" y="${arm_base_width}" z="${arm_base_height}"
+        <xacro:box_inertia m="0.5" x="${arm_base_length}" y="${arm_base_width}" z="${arm_base_height}"
                            o_xyz="0 0 ${arm_base_height / 2.0}" o_rpy="0 0 0" />
     </link>

File: src/my_robot_description/urdf/my_robot.urdf.xacro (robot description, xacro)
@@ -4,4 +4,11 @@
     <xacro:include filename="mobile_base.xacro" />
     <xacro:include filename="mobile_base_gazebo.xacro" />
+    <xacro:include filename="arm.xacro" />
+    <xacro:include filename="arm_gazebo.xacro" />
     <xacro:include filename="camera.xacro" />
+    <joint name="mobile_base_arm_joint" type="fixed">
+        <parent link="base_link" />
+        <child link="arm_base_link" />
+        <origin xyz="${base_length / 4.0} 0 ${base_height}" rpy="0 0 0" />
+    </joint>
 </robot>
